Commit message: Update pioneer3dx.urdf

File: urdf/pioneer3dx.urdf (robot description, URDF)
Before this commit: robot /home/leanhchien/catkin_ws/src/webots_ros/urdf/Pioneer3dx.urdf, 23 links, 22 joints
Links:
- removed link Hokuyo URG-04LX
- removed link IMU
- removed link so0
- removed link so1
- removed link so10
- removed link so11
- removed link so12
- removed link so13
- removed link so14
- removed link so15
- removed link so2
- removed link so3
- removed link so4
- removed link so5
- removed link so6
- removed link so7
- removed link so8
- removed link so9
- added link IU; collision box size=0.05 0.05 0.02; visual box size=0.05 0.05 0.02
- added link Lidar; collision box size=0.05 0.07 0.05; visual box size=0.05 0.07 0.05
- added link gps; collision cylinder length=0.05 radius=0.02; visual cylinder length=0.05 radius=0.02
Joints:
- removed joint base_link_Hokuyo URG-04LX_joint
- removed joint base_link_IMU_joint
- removed joint base_link_so0_joint
- removed joint base_link_so10_joint
- removed joint base_link_so11_joint
- removed joint base_link_so12_joint
- removed joint base_link_so13_joint
- removed joint base_link_so14_joint
- removed joint base_link_so15_joint
- removed joint base_link_so1_joint
- removed joint base_link_so2_joint
- removed joint base_link_so3_joint
- removed joint base_link_so4_joint
- removed joint base_link_so5_joint
- removed joint base_link_so6_joint
- removed joint base_link_so7_joint
- removed joint base_link_so8_joint
- removed joint base_link_so9_joint
- removed joint right wheel
- added joint base_link_IU_joint: type fixed, parent base_link, child IU, origin xyz=-0.06 0 0.15 rpy=0 0 0
- added joint base_link_Lidar_joint: type fixed, parent base_link, child Lidar, origin xyz=0.1 0 0.195 rpy=0 0 0
- added joint base_link_gps_joint: type fixed, parent base_link, child gps, origin xyz=0 0 0 rpy=0 0 0

Commit message: Update pioneer3dx.urdf

File: urdf/pioneer3dx.urdf (robot description, URDF)
Before this commit: robot /home/leanhchien/webots_ws/src/slam_pioneer3dx/urdf/pioneer3dx.urdf, 8 links, 6 joints
Joints:
- added joint right wheel: type continuous, parent base_link, child right wheel, origin xyz=0 -0.165 0 rpy=1.570796 0 -1.570796, axis -1 0 0, limit effort=10 velocity=12.3
